File: uBOT_v3_kicad_PCB/Micro_stepper_robot.kicad_pcb (KiCad board)
At the start: 2 copper layers, 37 x 47 mm, 29 parts, among them J4 USB_B_Mini, M1 Stepper_Motor_bipolar, M2 Stepper_Motor_bipolar, M3 Stepper_Motor_bipolar, M4 Stepper_Motor_bipolar, SW3 EN, SW4 BOOT, U1 DRV8833PW, U2 TCRT5000, U4 ESP32-WROOM-32D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

Commit message: progressed layout
Parts:
- M1, M2, M3, M4: moved to B.Cu

Commit message: routing 75% completed
Parts:
- J4: value USB_B_Mini -> USB_B_Micro; footprint Connector_USB:USB_Mini-B_Wuerth_65100516121_Horizontal -> Connector_USB:USB_Micro-B_Molex-105133-0001
- moved BT1 128.3 mm to (106.7, 75.9), turned to 270 degrees
- moved C4 125.3 mm to (105.7, 69.6)
- moved C5 124.2 mm to (105.7, 66.8)
- moved D1 119.1 mm to (106.7, 86.9)
- moved R6 117.0 mm to (106.7, 89.7)
- moved SW4 114.1 mm to (106.6, 83.6)
- moved R3 113.8 mm to (122.2, 67.6), turned to 90 degrees
- moved R4 110.0 mm to (124.7, 67.6), turned to 90 degrees
- moved R5 107.7 mm to (130.6, 56.6), turned to 90 degrees
- moved C3 102.3 mm to (123.2, 74.4), turned to 90 degrees
- moved C2 97.4 mm to (105.7, 64.0)
- moved C6 94.1 mm to (136.9, 73.7)
- moved R2 92.1 mm to (136.6, 89.9)
- moved R1 87.3 mm to (136.9, 81.8)
- moved R7 86.3 mm to (114.3, 60.7)
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
Commit message: routing completed :D
Parts:
- moved R6 30.4 mm to (113.3, 59.9)
- moved D1 29.9 mm to (113.4, 57.8)
- moved C5 23.8 mm to (129.2, 62.7), turned to 270 degrees
- moved C3 13.7 mm to (136.3, 78.5), turned to 0 degrees
- moved C1 13.5 mm to (123.4, 78.0)
- moved C2 10.4 mm to (111.1, 72.9), turned to 270 degrees
- moved C4 9.17 mm to (111.1, 77.0), turned to 270 degrees
- moved R7 8.76 mm to (105.5, 61.0), turned to 180 degrees
- moved U5 1.46 mm to (113.6, 55.0)
- moved R2 0.28 mm to (136.4, 90.0)
- turned SW4 to 180 degrees
Connections:
- U4 pad 14: Net-(U4-Pad14) -> /RIGHT_FAULT
- U4 pad 21: Net-(U4-Pad21) -> /MOTOR_SLEEP
- U4 pad 27: /MOTOR_SLEEP -> Net-(U4-Pad27)
- U4 pad 30: /RIGHT_FAULT -> Net-(U4-Pad30)
Routing:
- net +3V3: track 0.00 -> 101.3 mm
- net /LEFT_C: track 0.00 -> 87.1 mm, vias 0 -> 1
- net /LEFT_A: track 0.00 -> 74.0 mm, vias 0 -> 1
- net /IR_VOUT: track 0.00 -> 69.1 mm, vias 0 -> 2
- net +BATT: track 0.00 -> 67.7 mm
- net /LEFT_D: track 0.00 -> 62.3 mm, vias 0 -> 1
- net /LEFT_B: track 0.00 -> 57.9 mm, vias 0 -> 1
- net /RIGHT_D: track 0.00 -> 56.6 mm, vias 0 -> 2
- net /RIGHT_C: track 0.00 -> 53.2 mm, vias 0 -> 2
- net /MOTOR_SLEEP: track 0.00 -> 51.8 mm, vias 0 -> 2
- net /RIGHT_A: track 0.00 -> 48.8 mm, vias 0 -> 2
- net /RIGHT_B: track 0.00 -> 48.3 mm, vias 0 -> 2
- net /LEFT_D_IO: track 0.00 -> 30.2 mm, vias 0 -> 2
- net /LEFT_C_IO: track 0.00 -> 29.8 mm, vias 0 -> 2
- net +5V: track 0.00 -> 24.3 mm
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- added copper zone on B.Cu, net GND
- added copper zone on F.Cu, net GND
Other:
- net class Default: clearance 0.2 -> 0.1; trace_width 0.25 -> 0.1
- rule trace_clearance: 0.2 -> 0.1
- rule trace_min: 0.2 -> 0.1
- rule via_min_size: 0.4 -> 0.2
