File: uBOT_v3_kicad_PCB/Micro_stepper_robot.sch (KiCad schematic (older format))
At the start: 29 parts, among them J4 USB_B_Mini, M1 Stepper_Motor_bipolar, M2 Stepper_Motor_bipolar, M3 Stepper_Motor_bipolar, M4 Stepper_Motor_bipolar, SW3 EN, SW4 BOOT, U1 DRV8833PW, U2 TCRT5000, U4 ESP32-WROOM-32D, U5 MCP73812T-420I-OT, U6 FT231XS, U7 LM1117-3.3, U9 DRV8833PW

Commit message: finished assigning footprints, started layout
Parts:
- BT1: footprint (none) -> Connector_Molex:Molex_PicoBlade_53398-0271_1x02-1MP_P1.25mm_Vertical
- C1, C2, C3, C4, C5, C6: footprint (none) -> Capacitor_SMD:C_0805_2012Metric_Pad1.15x1.40mm_HandSolder
- D1: footprint (none) -> LED_SMD:LED_0603_1608Metric
- J4: footprint (none) -> Connector_USB:USB_Mini-B_Wuerth_65100516121_Horizontal
- R1, R3, R4, R5, R6, R7: footprint (none) -> Resistor_SMD:R_0805_2012Metric_Pad1.15x1.40mm_HandSolder
- R2: footprint Resistor_SMD:R_0805_2012Metric -> Resistor_SMD:R_0805_2012Metric_Pad1.15x1.40mm_HandSolder
- U2: footprint OPTO_TCRT5000 -> kicad_footprints:OPTO_TCRT5000
- U7: footprint (none) -> Package_TO_SOT_SMD:SOT-223-3_TabPin2
Changed lines of the file:
@@
 F 0 "BT1" H 2518 1246 50  0000 L CNN
 F 1 "Battery_Cell" H 2518 1155 50  0000 L CNN
-F 2 "" V 2400 1210 50  0001 C CNN
+F 2 "Connector_Molex:Molex_PicoBlade_53398-0271_1x02-1MP_P1.25mm_Vertical" V 2400 1210 50  0001 C CNN
 F 3 "~" V 2400 1210 50  0001 C CNN
 	1    2400 1150
@@
 F 0 "J4" H 7457 1667 50  0000 C CNN
 F 1 "USB_B_Mini" H 7457 1576 50  0000 C CNN
-F 2 "" H 7550 1150 50  0001 C CNN
+F 2 "Connector_USB:USB_Mini-B_Wuerth_65100516121_Horizontal" H 7550 1150 50  0001 C CNN
 F 3 "~" H 7550 1150 50  0001 C CNN
 	1    7400 1200
@@
 F 0 "U7" H 6050 1292 50  0000 C CNN
 F 1 "LM1117-3.3" H 6050 1201 50  0000 C CNN
-F 2 "" H 6050 1050 50  0001 C CNN
+F 2 "Package_TO_SOT_SMD:SOT-223-3_TabPin2" H 6050 1050 50  0001 C CNN
 F 3 "http://www.ti.com/lit/ds/symlink/lm1117.pdf" H 6050 1050 50  0001 C CNN
 	1    6050 1050
@@
 F 0 "R3" V 7704 1200 50  0000 C CNN
 F 1 "27R" V 7795 1200 50  0000 C CNN
-F 2 "" H 7900 1200 50  0001 C CNN
+F 2 "Resistor_SMD:R_0805_2012Metric_Pad1.15x1.40mm_HandSolder" H 7900 1200 50  0001 C CNN
 F 3 "~" H 7900 1200 50  0001 C CNN
 	1    7900 1200
@@
 F 0 "R4" V 8100 1300 50  0000 C CNN
 F 1 "27R" V 8000 1300 50  0000 C CNN
-F 2 "" H 7900 1300 50  0001 C CNN
+F 2 "Resistor_SMD:R_0805_2012Metric_Pad1.15x1.40mm_HandSolder" H 7900 1300 50  0001 C CNN
 F 3 "~" H 7900 1300 50  0001 C CNN
 	1    7900 1300
@@
 F 0 "R2" V 743 2350 50  0000 C CNN
 F 1 "10K" V 834 2350 50  0000 C CNN
-F 2 "Resistor_SMD:R_0805_2012Metric" V 880 2350 50  0001 C CNN
+F 2 "Resistor_SMD:R_0805_2012Metric_Pad1.15x1.40mm_HandSolder" V 880 2350 50  0001 C CNN
 F 3 "~" H 950 2350 50  0001 C CNN
 	1    950  2350
@@
 F 0 "C4" H 9908 4104 50  0000 R CNN
 F 1 "C_Small" H 9908 4195 50  0000 R CNN
-F 2 "" H 10000 4150 50  0001 C CNN
+F 2 "Capacitor_SMD:C_0805_2012Metric_Pad1.15x1.40mm_HandSolder" H 10000 4150 50  0001 C CNN
 F 3 "~" H 10000 4150 50  0001 C CNN
 	1    10000 4150
@@
 F 0 "C2" V 8950 4600 50  0000 C CNN
 F 1 "0.01uF" V 9050 4500 50  0000 C CNN
-F 2 "" H 9000 4700 50  0001 C CNN
+F 2 "Capacitor_SMD:C_0805_2012Metric_Pad1.15x1.40mm_HandSolder" H 9000 4700 50  0001 C CNN
 F 3 "~" H 9000 4700 50  0001 C CNN
 	1    9000 4700
@@
 F 0 "C3" H 9908 1604 50  0000 R CNN
 F 1 "C_Small" H 9908 1695 50  0000 R CNN
-F 2 "" H 10000 1650 50  0001 C CNN
+F 2 "Capacitor_SMD:C_0805_2012Metric_Pad1.15x1.40mm_HandSolder" H 10000 1650 50  0001 C CNN
 F 3 "~" H 10000 1650 50  0001 C CNN
 	1    10000 1650
@@
 F 0 "C1" V 8950 2100 50  0000 C CNN
 F 1 "0.01uF" V 9050 2000 50  0000 C CNN
-F 2 "" H 9000 2200 50  0001 C CNN
+F 2 "Capacitor_SMD:C_0805_2012Metric_Pad1.15x1.40mm_HandSolder" H 9000 2200 50  0001 C CNN
 F 3 "~" H 9000 2200 50  0001 C CNN
 	1    9000 2200
@@
 F 0 "U2" H 1400 1465 50  0000 C CNN
 F 1 "TCRT5000" H 1400 1374 50  0000 C CNN
-F 2 "OPTO_TCRT5000" H 1400 1100 50  0001 L BNN
+F 2 "kicad_footprints:OPTO_TCRT5000" H 1400 1100 50  0001 L BNN
 F 3 "Vishay" H 1400 1100 50  0001 L BNN
 F 4 "7.2mm" H 1400 1100 50  0001 L BNN "Field4"
@@
 F 0 "R1" H 1159 1496 50  0000 L CNN
 F 1 "10k" H 1159 1405 50  0000 L CNN
-F 2 "" H 1100 1450 50  0001 C CNN
+F 2 "Resistor_SMD:R_0805_2012Metric_Pad1.15x1.40mm_HandSolder" H 1100 1450 50  0001 C CNN
 F 3 "~" H 1100 1450 50  0001 C CNN
 	1    1100 1450
@@
 F 0 "R5" H 1759 1496 50  0000 L CNN
 F 1 "220R" H 1759 1405 50  0000 L CNN
-F 2 "" H 1700 1450 50  0001 C CNN
+F 2 "Resistor_SMD:R_0805_2012Metric_Pad1.15x1.40mm_HandSolder" H 1700 1450 50  0001 C CNN
 F 3 "~" H 1700 1450 50  0001 C CNN
 	1    1700 1450
@@
 F 0 "C5" V 4429 750 50  0000 C CNN
 F 1 "4.7uF" V 4338 750 50  0000 C CNN
-F 2 "" H 4200 750 50  0001 C CNN
+F 2 "Capacitor_SMD:C_0805_2012Metric_Pad1.15x1.40mm_HandSolder" H 4200 750 50  0001 C CNN
 F 3 "~" H 4200 750 50  0001 C CNN
 	1    4200 750
@@
 F 0 "D1" H 3700 1085 50  0000 C CNN
 F 1 "LED_Small" H 3700 994 50  0000 C CNN
-F 2 "" V 3700 850 50  0001 C CNN
+F 2 "LED_SMD:LED_0603_1608Metric" V 3700 850 50  0001 C CNN
 F 3 "~" V 3700 850 50  0001 C CNN
 	1    3700 850
@@
 F 0 "R6" H 3300 1050 50  0000 L CNN
 F 1 "220R" H 3200 950 50  0000 L CNN
-F 2 "" H 3450 1000 50  0001 C CNN
+F 2 "Resistor_SMD:R_0805_2012Metric_Pad1.15x1.40mm_HandSolder" H 3450 1000 50  0001 C CNN
 F 3 "~" H 3450 1000 50  0001 C CNN
 	1    3450 1000
@@
 F 0 "R7" H 3450 1500 50  0000 L CNN
 F 1 "2k" H 3450 1400 50  0000 L CNN
-F 2 "" H 3600 1450 50  0001 C CNN
+F 2 "Resistor_SMD:R_0805_2012Metric_Pad1.15x1.40mm_HandSolder" H 3600 1450 50  0001 C CNN
 F 3 "~" H 3600 1450 50  0001 C CNN
 	1    3600 1450
@@
 F 0 "C6" V 4929 1200 50  0000 C CNN
 F 1 "4.7uF" V 4838 1200 50  0000 C CNN
-F 2 "" H 4700 1200 50  0001 C CNN
+F 2 "Capacitor_SMD:C_0805_2012Metric_Pad1.15x1.40mm_HandSolder" H 4700 1200 50  0001 C CNN
 F 3 "~" H 4700 1200 50  0001 C CNN
 	1    4700 1200

Commit message: completed rough footprint placement
Parts:
- J4: value USB_B_Mini -> USB_B_Micro; footprint Connector_USB:USB_Mini-B_Wuerth_65100516121_Horizontal -> Connector_USB:USB_Micro-B_Molex-105133-0001
Changed lines of the file:
@@
 P 7400 1200
 F 0 "J4" H 7457 1667 50  0000 C CNN
-F 1 "USB_B_Mini" H 7457 1576 50  0000 C CNN
-F 2 "Connector_USB:USB_Mini-B_Wuerth_65100516121_Horizontal" H 7550 1150 50  0001 C CNN
+F 1 "USB_B_Micro" H 7457 1576 50  0000 C CNN
+F 2 "Connector_USB:USB_Micro-B_Molex-105133-0001" H 7550 1150 50  0001 C CNN
 F 3 "~" H 7550 1150 50  0001 C CNN
 	1    7400 1200

Commit message: routing completed :D
Connections:
- net MOTOR_SLEEP: now also U4.21 (SDO/SD0); no longer U4.27 (IO16)
- net RIGHT_FAULT: now also U4.14 (IO12); no longer U4.30 (IO18)
Changed lines of the file:
@@
 	1    0    0    -1
 $EndComp
-Text Label 2750 3650 0    50   ~ 0
+Text Label 1450 3850 2    50   ~ 0
 MOTOR_SLEEP
-Wire Wire Line
-	2700 3650 2750 3650
 Text Label 9100 4600 2    50   ~ 0
 MOTOR_SLEEP
@@
 Wire Wire Line
 	9850 1300 10450 1300
-Text Label 2750 3750 0    50   ~ 0
-LEFT_FAULT
-Text Label 2750 3850 0    50   ~ 0
+Text Label 2750 3250 0    50   ~ 0
 RIGHT_FAULT
-Wire Wire Line
-	2700 3750 2750 3750
-Wire Wire Line
-	2700 3850 2750 3850
 Text Notes 8700 4250 0    100  ~ 0
 LEFT MOTORS
@@
 	4300 750  4950 750
 Connection ~ 4950 1200
+Wire Wire Line
+	2700 3250 2750 3250
+Wire Wire Line
+	2700 3750 2750 3750
+Text Label 2750 3750 0    50   ~ 0
+LEFT_FAULT
+Wire Wire Line
+	1450 3850 1500 3850
 $EndSCHEMATC
